File: MegaBiels.kicad_pcb (KiCad board)
At the start: 2 copper layers, 150 x 30 mm, 4 parts

Commit message: Added OSHW logo
Parts:
- added G***: LOGO, w_logo:Logo_copper_OSHW_12x13mm, B.Cu at (169.5, 60.0)
